Commit message: Update: project 4 Map my world

File: src/my_robot/urdf/my_robot.xacro (robot description, xacro)
@@ -177,3 +177,10 @@
     <dynamics damping="1.0" friction="1.0"/>
   </joint>
+  <joint name="camera_optical_joint" type="fixed">
+    <origin xyz="0 0 0" rpy="-1.5707 0 -1.5707"/>
+    <parent link="camera"/>
+    <child link="camera_optical"/>
+  </joint>
+  <link name="camera_optical">
+  </link>
 </robot>
